File: APRL/APRL.kicad_pcb (KiCad board)
At the start: 2 copper layers, 1 part, among them U1 BMP581

Commit message: schematics
Parts:
- removed U1: BMP581, footprints:QFN10_BMP581_BOS
- added 3.3V: AP1117-15, Package_TO_SOT_SMD:SOT-223-3_TabPin2, F.Cu at (140.3, 111.5)
- added 3.3V: LED, LED_SMD:LED_0603_1608Metric, F.Cu at (122.0, 131.5)
- added 5V: AP1117-50, Package_TO_SOT_SMD:SOT-223-3_TabPin2, F.Cu at (140.4, 120.7)
- added 5V: LED, LED_SMD:LED_0603_1608Metric, F.Cu at (122.1, 135.0)
- added BAT1: BS-7, footprints:Battery_Holder_Coin_2032_BS-7, F.Cu at (128.3, 94.2)
- added BT1: 2S, footprints:AMASS_XT30PW-M_1x02_P2.50mm_Horizontal, F.Cu at (136.5, 131.2)
- added Baro: BMP581, footprints:QFN10_BMP581_BOS, F.Cu at (171.9, 108.2)
- added C1: 22uF, Capacitor_SMD:C_0805_2012Metric, F.Cu at (127.0, 125.7)
- added C10: 10uF, Capacitor_SMD:C_0603_1608Metric, F.Cu at (137.4, 116.0)
- added C11: 100uF, Capacitor_SMD:C_0805_2012Metric, F.Cu at (146.4, 113.3)
- added C12: 2.2uF, Capacitor_SMD:C_0603_1608Metric, F.Cu at (143.2, 99.0)
- added C13: 100nF, Capacitor_SMD:C_0603_1608Metric, F.Cu at (146.5, 101.2)
- added C14: 100nF, Capacitor_SMD:C_0603_1608Metric, F.Cu at (141.4, 101.8)
- added C15: 4.7 uF, Capacitor_SMD:C_0603_1608Metric, F.Cu at (155.1, 61.9)
- added C16: 100nF, Capacitor_SMD:C_0603_1608Metric, F.Cu at (154.0, 54.9)
- added C2: 100nF, Capacitor_SMD:C_0603_1608Metric, F.Cu at (168.4, 99.2)
- added C3: 10uF, Capacitor_SMD:C_0805_2012Metric, F.Cu at (123.5, 125.8)
- added C4: 100nF, Capacitor_SMD:C_0805_2012Metric, F.Cu at (119.8, 125.7)
- added C5: 100nF, Capacitor_SMD:C_0603_1608Metric, F.Cu at (175.2, 98.5)
- added C6: 100nF, Capacitor_SMD:C_0603_1608Metric, F.Cu at (174.9, 108.1)
- added C7: 100nF, Capacitor_SMD:C_0603_1608Metric, F.Cu at (172.0, 110.8)
- added C8: 1 uF, Capacitor_SMD:C_0603_1608Metric, F.Cu at (137.6, 125.5)
- added C9: 100 nF, Capacitor_SMD:C_0603_1608Metric, F.Cu at (145.8, 125.5)
- added G***: LOGO, LOGO, B.Cu at (126.8, 64.6)
- added G***: LOGO, LOGO, B.Cu at (165.5, 67.6)
- added GPS1: CAM-M8C-0, footprints:QFN_M8C-0_UBL, F.Cu at (146.7, 55.9)
- added I/O: Conn_01x05_Pin, Connector_PinHeader_2.54mm:PinHeader_1x05_P2.54mm_Vertical, F.Cu at (144.5, 71.2)
- added I2C: Conn_01x02_Pin, Connector_PinHeader_2.54mm:PinHeader_1x02_P2.54mm_Vertical, F.Cu at (172.2, 116.3)
- added IMU: BMI088, footprints:PQFN50P450X300X100-16N, F.Cu at (171.7, 99.8)
- added J1: Conn_01x03_Pin, Connector_PinHeader_2.54mm:PinHeader_1x03_P2.54mm_Vertical, F.Cu at (138.1, 58.5)
- added Lora: E22-900M22S, footprints:E22-900M22S, F.Cu at (124.3, 113.7)
- added MCU1: Teensy 4.1, footprints:Teensy_41, F.Cu at (157.1, 104.9)
- added Mag: BMM350, footprints:BGA9_BMM350_BOS, F.Cu at (143.7, 101.3)
- added R1: 1k, Resistor_SMD:R_0603_1608Metric, F.Cu at (118.6, 135.0)
- added R2: 1k, Resistor_SMD:R_0603_1608Metric, F.Cu at (118.5, 131.4)
- added R3: 1k, Resistor_SMD:R_0603_1608Metric, F.Cu at (170.8, 134.1)
- added REF**: MountingHole_3.2mm_M3_Pad_Via, MountingHole:MountingHole_3.2mm_M3_Pad_Via, F.Cu at (126.8, 54.5)
- added REF**: MountingHole_3.2mm_M3_Pad_Via, MountingHole:MountingHole_3.2mm_M3_Pad_Via, F.Cu at (126.8, 140.0)
- added REF**: MountingHole_3.2mm_M3_Pad_Via, MountingHole:MountingHole_3.2mm_M3_Pad_Via, F.Cu at (166.8, 54.5)
- added REF**: MountingHole_3.2mm_M3_Pad_Via, MountingHole:MountingHole_3.2mm_M3_Pad_Via, F.Cu at (166.8, 140.0)
- added SPI: Conn_01x03_Pin, Connector_PinHeader_2.54mm:PinHeader_1x03_P2.54mm_Vertical, F.Cu at (171.2, 79.3)
- added SPI1: Conn_01x03_Pin, Connector_PinHeader_2.54mm:PinHeader_1x03_P2.54mm_Vertical, F.Cu at (171.1, 89.5)
- added Status: LED, LED_SMD:LED_0603_1608Metric, F.Cu at (174.1, 134.1)
Routing:
- net +3.3V: track 0.00 -> 202.1 mm, vias 0 -> 4
- net SPI_MISO1: track 0.00 -> 117.7 mm, vias 0 -> 1
- net SPI_MOSI1: track 0.00 -> 113.7 mm, vias 0 -> 1
- net SPI_SCK1: track 0.00 -> 95.1 mm, vias 0 -> 1
- net SPI_SCK: track 0.00 -> 76.0 mm
- net +5V: track 0.00 -> 49.6 mm
- net SCL: track 0.00 -> 40.7 mm
- net SDA: track 0.00 -> 37.9 mm
- net /DIO2: track 0.00 -> 36.5 mm, vias 0 -> 1
- net RXEN: track 0.00 -> 35.7 mm, vias 0 -> 1
- net SPI_MISO: track 0.00 -> 34.9 mm
- net TXEN: track 0.00 -> 34.7 mm, vias 0 -> 1
- net Net-(GPS1-V_BCKP): track 0.00 -> 32.9 mm, vias 0 -> 1
- net IMU_INT1: track 0.00 -> 31.5 mm, vias 0 -> 1
- net SPI_MOSI: track 0.00 -> 25.0 mm, vias 0 -> 1
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- added copper zone on B.Cu, net GND
- added copper zone on F.Cu, net GND
Other:
- board outline added: 61 x 96.2 mm
- board text added: "-+"
- board text added: "34 35 36 37 38"
- board text added: "APRL Avionics Ver 1.0"
- board text added: "APRL Gliding Beaver"
- board text added: "Barometer: BMI088 Lora : E22-900M22S Magnet. : BMM350 GPS : CAM-M8C-0 IMU : BMI088 MCU : Teensy 4.1"
- board text added: "D_Sel"
- board text added: "IMU"
- board text added: "Reset"
- board text added: "SCK MISO MOSI"
- board text added: "SDA SCL"
- board text added: "Safeboot"

Commit message: revision 1 of avionics board
Parts:
- removed the G*** at (165.5, 67.6)
- added SW1: SW_SPST, footprints:slide_sw, F.Cu at (140.6, 129.5)
- BT1: footprint footprints:AMASS_XT30PW-M_1x02_P2.50mm_Horizontal -> Connector_JST:JST_PH_S2B-PH-K_1x02_P2.00mm_Horizontal
- C4: footprint Capacitor_SMD:C_0805_2012Metric -> Capacitor_SMD:C_0603_1608Metric
- J1: value Conn_01x03_Pin -> Conn_01x02_Pin; footprint Connector_PinHeader_2.54mm:PinHeader_1x03_P2.54mm_Vertical -> Connector_PinHeader_2.54mm:PinHeader_1x02_P2.54mm_Vertical
- moved C12 35.6 mm to (118.7, 73.2)
- moved C13 35.6 mm to (122.0, 75.4)
- moved Mag1 35.6 mm to (119.3, 75.4)
- moved C14 35.6 mm to (117.0, 75.9)
- moved BT1 12.8 mm to (147.4, 137.9), turned to 0 degrees
- moved J2 7.32 mm to (142.5, 78.2)
- moved BAT1 3.48 mm to (127.5, 97.6)
- moved C8 3.31 mm to (135.1, 123.3), turned to 180 degrees
- moved J1 1.19 mm to (138.7, 57.4), turned to 0 degrees
- moved 5V1 0.90 mm to (141.3, 120.6)
- renumbered 3.3V to 3.3V1, 5V to 5V1, Baro to Baro1, 5V to D1, 3.3V to D2, Status to D3, I2C to I2C1, IMU to IMU1, I/O to J2, Lora to Lora1, Mag to Mag1, SPI to SPI_1
Connections:
- net IMU_CSB1 renamed ACCEL_CS
- BT1 pad 2: Net-(5V1-VI) -> Net-(BT1--)
- GPS1 pad 20: Net-(GPS1-D_SEL) -> GND
- GPS1 pad 3: CAM_CS -> GPS_CS
- IMU1 pad 1: unconnected-(IMU1-INT2-Pad1) -> /IMU_INT2
- IMU1 pad 12: IMU_INT3 -> Net-(IMU1-INT1)
- IMU1 pad 16: IMU_INT1 -> Net-(IMU1-INT1)
- IMU1 pad 5: IMU_CSB2 -> GYRO_CS
- J1 pad 1: Net-(GPS1-SAFEBOOT_N) -> Net-(GPS1-RESET_N)
- J1 pad 2: Net-(GPS1-RESET_N) -> Net-(GPS1-SAFEBOOT_N)
- MCU1 pad 29: IMU_INT3 -> /IMU_INT2
- MCU1 pad 31: unconnected-(MCU1-CTX3-Pad31) -> GYRO_CS
- MCU1 pad 32: IMU_INT1 -> GPS_CS
Routing:
- net /IMU_INT2: track 0.00 -> 44.9 mm, vias 0 -> 1
- net SDA: track 37.9 -> 82.1 mm
- net +3.3V: track 202.1 -> 245.3 mm, vias 4 -> 8
- net SCL: track 40.7 -> 80.4 mm
- net MAG_INT: track 10.1 -> 42.1 mm, vias 1 -> 0
- net IMU_INT1: track 31.5 -> 0.00 mm, vias 1 -> 0
- net GYRO_CS: track 0.00 -> 27.7 mm, vias 0 -> 1
- net GPS_CS: track 0.00 -> 25.1 mm
- net IMU_INT3: track 19.3 -> 0.00 mm, vias 1 -> 0
- net GND: track 18.1 -> 30.2 mm, vias 212 -> 279
- net Net-(BT1--): track 0.00 -> 10.8 mm
- net SPI_MOSI1: track 113.7 -> 105.5 mm
- net Net-(IMU1-INT1): track 0.00 -> 6.02 mm, vias 0 -> 2
- net SPI_MISO1: track 117.7 -> 111.9 mm
- net Net-(GPS1-D_SEL): track 4.50 -> 0.00 mm
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Other:
- board size 61 x 96.2 mm -> 61.8 x 96.2 mm
- board text added: "+"
- board text added: "-"
- board text added: "APRL Avionics Ver 1.1"
- board text added: "Barometer: BMP581 Lora : E22-900M22S Magnet. : BMM350 GPS : CAM-M8C-0 IMU : BMI088 MCU : Teensy 4.1"
- board text added: "HB"
- board text added: "Obsidian Gorilla"
- board text added: "X"
- board text added: "Y"
- board text added: "Z"
- board text removed: "-+"
- board text removed: "APRL Avionics Ver 1.0"
- board text removed: "APRL Gliding Beaver"
- board text removed: "Barometer: BMI088 Lora : E22-900M22S Magnet. : BMM350 GPS : CAM-M8C-0 IMU : BMI088 MCU : Teensy 4.1"
- board text removed: "D_Sel"
