File: APRL/APRL.kicad_sch (KiCad schematic)
At the start: 17 parts, among them U1 BMP581, U2 BMM350

Commit message: schematics
Parts:
- removed 5V_REG: LM7805_TO220, Package_TO_SOT_THT:TO-220-3_Vertical, symbol Regulator_Linear:LM7805_TO220
- removed MCU: TEENSY_4.1, footprints:TEENSY_LONG_EXT, symbol TEENSY_4.1:TEENSY_4.1
- added 5V1: AP1117-50, Package_TO_SOT_SMD:SOT-223-3_TabPin2, symbol Regulator_Linear:AP1117-50
- added C1: 22uF, Capacitor_SMD:C_0805_2012Metric, symbol Device:C_Small
- added C12: 2.2uF, Capacitor_SMD:C_0603_1608Metric, symbol Device:C_Small
- added C14, C16, C2: 100nF, Capacitor_SMD:C_0603_1608Metric, symbol Device:C_Small
- added C15: 4.7 uF, Capacitor_SMD:C_0603_1608Metric, symbol Device:C_Small
- added C3: 10uF, Capacitor_SMD:C_0805_2012Metric, symbol Device:C_Small
- added C4: 100nF, Capacitor_SMD:C_0805_2012Metric, symbol Device:C_Small
- added D1, D2, D3: LED, LED_SMD:LED_0603_1608Metric, symbol Device:LED
- added GPS1: CAM-M8C-0, footprints:QFN_M8C-0_UBL, symbol 2024-02-02_03-39-15:CAM-M8C-0
- added I2C1: Conn_01x02_Pin, Connector_PinHeader_2.54mm:PinHeader_1x02_P2.54mm_Vertical, symbol Connector:Conn_01x02_Pin
- added J1, SPI1, SPI_1: Conn_01x03_Pin, Connector_PinHeader_2.54mm:PinHeader_1x03_P2.54mm_Vertical, symbol Connector:Conn_01x03_Pin
- added J2: Conn_01x05_Pin, Connector_PinHeader_2.54mm:PinHeader_1x05_P2.54mm_Vertical, symbol Connector:Conn_01x05_Pin
- added MCU1: Teensy 4.1, footprints:Teensy_41, symbol TEENSY_41:DEV-16771
- added R1, R2, R3: 1k, Resistor_SMD:R_0603_1608Metric, symbol Device:R_Small
- BAT1: footprint digikey-footprints:Battery_Holder_Coin_2032_BS-7 -> footprints:Battery_Holder_Coin_2032_BS-7
- BT1: footprint (none) -> footprints:AMASS_XT30PW-M_1x02_P2.50mm_Horizontal
- C10: renamed from C6; footprint (none) -> Capacitor_SMD:C_0603_1608Metric
- C11: renamed from C5; footprint (none) -> Capacitor_SMD:C_0805_2012Metric
- C13: renamed from C8; footprint (none) -> Capacitor_SMD:C_0603_1608Metric
- C5: renamed from C7; footprint (none) -> Capacitor_SMD:C_0603_1608Metric
- C6: renamed from C1; footprint (none) -> Capacitor_SMD:C_0603_1608Metric
- C7: renamed from C2; footprint (none) -> Capacitor_SMD:C_0603_1608Metric
- C8: renamed from C4; value 0.33uF -> 1 uF; footprint (none) -> Capacitor_SMD:C_0603_1608Metric
- C9: renamed from C3; value 0.1uF -> 100 nF; footprint (none) -> Capacitor_SMD:C_0603_1608Metric
- renumbered 3.3V_REG to 3.3V1, U1 to Baro1, IMU to IMU1, Lora to Lora1, U2 to Mag1
Connections:
- net GND: now also BAT1.Neg, BT1.1 (+), C5.1, IMU1.2 (NC), IMU1.4 (GNDA), IMU1.6 (GNDIO), IMU1.7 (PS), Mag1.B1 (GND), Mag1.B2 (ADSEL), Mag1.C3 (BYPASS), 5V1.1 (GND), C1.2, C12.2, C14.2, C15.2, C16.2, C2.2, C3.2, C4.2, D3.1 (K), GPS1.10 (GND), GPS1.11 (GND), GPS1.12 (GND), GPS1.13 (GND), GPS1.14 (GND), GPS1.15 (GND), GPS1.18 (GND), GPS1.19 (GND), GPS1.21 (GND), GPS1.22 (GND), GPS1.27 (GND), GPS1.31 (GND), GPS1.4 (GND), GPS1.5 (GND), MCU1.GND1 (GND), MCU1.GND2 (GND__1), MCU1.GND3 (GND__2), MCU1.GND4 (GND__3), MCU1.GND5 (GND__4), MCU1.USB_GND1 (USB_GND), MCU1.USB_GND2 (USB_GND__1), R1.2, R2.1; no longer BT1.2 (-), C5.2
- net SPI_MISO: now also IMU1.10 (SDO2), IMU1.15 (SDO1), MCU1.12 (MISO), SPI1.2 (Pin_2)
- net SPI_MOSI: now also IMU1.9 (SDA/SDI), MCU1.11 (MOSI), SPI1.3 (Pin_3)
- net SPI_SCK: now also IMU1.8 (SCL/SCK), MCU1.13 (SCK), SPI1.1 (Pin_1)
- net at C8.1: now also BT1.2 (-), 5V1.3 (VI); no longer BT1.1 (+)
- net CSB: now reaches Baro1.6 (CSB)
- net CSB: now also MCU1.10 (CS1)
- net INTB: now reaches Baro1.7 (INT)
- net INTB: now also MCU1.9 (OUT1C)
- net at BAT1.Pos: now also C16.1, GPS1.8 (V_BCKP)
- net +3.3V: now reaches IMU1.11 (VDDIO)
- net +3.3V: now also 3.3V1.2 (VO), Baro1.1 (VDDIO), Baro1.10 (VDD), C11.1, C13.1, C5.2, C6.1, C7.1, IMU1.3 (VDD), Lora1.9 (VCC), Mag1.B3 (VDDIO), Mag1.C1 (VDD), C1.1, C14.1, C15.1, C2.1, C3.1, C4.1, D2.2 (A), GPS1.1 (VCC_IO), GPS1.9 (VCC), MCU1.3.3V_1 (3.3V), MCU1.3.3V_2 (3.3V__1), MCU1.3.3V_3 (3.3V__2)
- net IMU_INT3: now reaches IMU1.12 (INT3)
- net IMU_INT3: now also MCU1.29 (TX7)
- net IMU_CSB1: now reaches IMU1.14 (CSB1)
- net IMU_CSB1: now also MCU1.30 (CRX3)
- net IMU_INT1: now reaches IMU1.16 (INT1)
- net IMU_INT1: now also MCU1.32 (OUT1B)
- net IMU_CSB2: now reaches IMU1.5 (CSB2)
- net +5V: now reaches 3.3V1.3 (VI), C10.1, C9.1
- net +5V: now also 5V1.2 (VO), D1.2 (A), MCU1.VIN
- net MAG_INT: now reaches Mag1.A1 (INT)
- net MAG_INT: now also MCU1.41 (A17)
- net SDA: now reaches Mag1.A2 (SDA)
- net SDA: now also I2C1.2 (Pin_2), MCU1.18 (A4)
- net SCL: now reaches Mag1.A3 (SCK)
- net SCL: now also I2C1.1 (Pin_1), MCU1.19 (A5)
- net at Mag1.C2 (CRST): now also C12.1
- net DIO1: now reaches Lora1.13 (DIO1)
- net DIO1: now also MCU1.17 (A3)
- net BUSY: now reaches Lora1.14 (BUSY)
- net BUSY: now also MCU1.16 (A2)
- net NRST: now reaches Lora1.15 (NRST)
- net NRST: now also MCU1.15 (A1)
- net SPI_MISO1: now reaches Lora1.16 (MISO)
- net SPI_MISO1: now also GPS1.25 (MISO), MCU1.39 (A15), SPI_1.2 (Pin_2)
- net SPI_MOSI1: now reaches Lora1.17 (MOSI)
- net SPI_MOSI1: now also GPS1.26 (MOSI), MCU1.26 (A12), SPI_1.3 (Pin_3)
- net SPI_SCK1: now reaches Lora1.18 (SCK)
- net SPI_SCK1: now also GPS1.6 (SCK), MCU1.27 (A13), SPI_1.1 (Pin_1)
- net NSS: now reaches Lora1.19 (NSS)
- net NSS: now also MCU1.14 (A0)
- net RXEN: now reaches Lora1.6 (RXEN)
- net RXEN: now also MCU1.20 (A6)
- net TXEN: now reaches Lora1.7 (TXEN)
- net TXEN: now also MCU1.21 (A7)
- net DIO2: now reaches Lora1.8 (DIO2)
- net DIO2: now also MCU1.23 (A9)
- new net: GPS1.24 (SAFEBOOT_N), J1.1 (Pin_1)
- new net: GPS1.23 (RESET_N), J1.2 (Pin_2)
- new net: GPS1.20 (D_SEL), J1.3 (Pin_3)
- new net: D2.1 (K), R2.2
- new net: D1.1 (K), R1.1
- new net: D3.2 (A), R3.1
- new net: MCU1.2 (OUT2), R3.2
- new net: GPS1.16 (RF_OUT), GPS1.17 (RF_IN)
- new net 34: J2.1 (Pin_1), MCU1.34 (RX8)
- new net 35: J2.2 (Pin_2), MCU1.35 (TX8)
- new net 36: J2.3 (Pin_3), MCU1.36 (CS2)
- new net 37: J2.4 (Pin_4), MCU1.37 (CS3)
- new net 38: J2.5 (Pin_5), MCU1.38 (A14)
- new net 5: MCU1.5 (IN2)
- new net CAM_CS: GPS1.3 (CS)
- new net PPS: GPS1.29 (PPS), MCU1.33 (MCLK2)
- no-connect marks 0 -> 32
Other:
- note added: "3.3V Regulator"
- note added: "5V Regulator"
- note added: "Barometer"
- note added: "Coin cell for RTC and GPS"
- note added: "Extra I/O"
- note added: "GPS Module- No RTK"
- note added: "I2C test point"
- note added: "Inertial Measurement Unit"
- note added: "Lipo 2s"
- note added: "Magnetometer"
- note added: "NSS chip select"
- note added: "Radio Transmitter"
- note added: "SPI Test Points"
- note added: "stamp hole 50Ω impedance"
- note added: "status led"
- company: (none) -> APRL
- title: (none) -> Avionics Board
- moved on the sheet: 3.3V1, BAT1, BT1, Baro1, C10, C11, C13, C5, C6, C7, C8, C9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

Commit message: revision 1 of avionics board
Parts:
- removed J1: Conn_01x03_Pin, Connector_PinHeader_2.54mm:PinHeader_1x03_P2.54mm_Vertical, symbol Connector:Conn_01x03_Pin
- added J1: Conn_01x02_Pin, Connector_PinHeader_2.54mm:PinHeader_1x02_P2.54mm_Vertical, symbol Connector:Conn_01x02_Pin
- added SW1: SW_SPST, footprints:slide_sw, symbol Switch:SW_SPST
- BT1: footprint footprints:AMASS_XT30PW-M_1x02_P2.50mm_Horizontal -> Connector_JST:JST_PH_S2B-PH-K_1x02_P2.00mm_Horizontal
- C4: footprint Capacitor_SMD:C_0805_2012Metric -> Capacitor_SMD:C_0603_1608Metric
Connections:
- net IMU_CSB2 is gone; now on net GYRO_CS: IMU1.5 (CSB2)
- net GND: now also GPS1.20 (D_SEL)
- net at GPS1.24 (SAFEBOOT_N): now also J1.2 (Pin_2)
- net at GPS1.23 (RESET_N): now also J1.1 (Pin_1)
- net at 5V1.3 (VI), C8.1: now also SW1.2 (B); no longer BT1.2 (-)
- net IMU_INT2: now reaches IMU1.1 (INT2)
- net IMU_INT2: now also MCU1.29 (TX7)
- net GYRO_CS: now reaches MCU1.31 (CTX3)
- net CAM_CS renamed GPS_CS
- net GPS_CS: now also MCU1.32 (OUT1B)
- net IMU_CSB1 renamed ACCEL_CS
- net IMU_INT1: no longer names the net of IMU1.16 (INT1)
- net IMU_INT1: now also IMU1.12 (INT3); no longer MCU1.32 (OUT1B)
- removed net IMU_INT3: IMU1.12 (INT3), MCU1.29 (TX7)
- new net: BT1.2 (-), SW1.1 (A)
- no-connect marks 32 -> 30
Other:
- note added: "D_SEL to GND for SPI mode"
- note added: "NSS == chip select"
- note added: "SPI1 = SPI SPI_1 = SPI 1"
- note added: "Sync. mode for accel and gyro"
- note removed: "NSS chip select"
- moved on the sheet: 3.3V1, 5V1, C1, C10, C11, C3, C4, C8, C9, D1, D2, Lora1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
